File: PCB/Nexus Hackpad.kicad_pcb (KiCad board)
At the start: 2 copper layers, 70 x 100 mm, 32 parts, among them SW1 SW_Push, SW10 RotaryEncoder_Switch, SW2 SW_Push, SW3 SW_Push, SW4 SW_Push, SW5 SW_Push, SW6 SW_Push, SW7 SW_Push, SW8 SW_Push, SW9 SW_Push, U1 MOUDLE-SEEEDUINO-XIAO, U2 ER_OLEDM0.91_1x-I2C

Commit message: Merge branches 'main' and 'main' of https://github.com/ttayG-sr/Nexus-Hackpad
Connections:
- net /GND renamed GND
- D10 pad 1: /3V3 -> +5V
- D11 pad 1: /3V3 -> +5V
- D12 pad 1: /3V3 -> +5V
- D13 pad 1: /3V3 -> +5V
- D14 pad 1: /3V3 -> +5V
- D15 pad 1: /3V3 -> +5V
- D16 pad 1: /3V3 -> +5V
- D17 pad 1: /3V3 -> +5V
- D18 pad 1: /3V3 -> +5V
- U1 pad 12: /3V3 -> +3V3
- U1 pad 14: unconnected-(U1-5V-Pad14) -> +5V
- U2 pad 2: /3V3 -> +3V3
Routing:
- net +5V: track 0.00 -> 266.3 mm, vias 0 -> 9
- net /3V3: track 264.8 -> 0.00 mm, vias 9 -> 0
- net +3V3: track 0.00 -> 36.0 mm
